Commit message: 1 5 6

File: src/ur5e_gripper/urdf/ur5e_with_gripper.urdf (robot description, URDF)
Before this commit: robot ur5e_with_gripper, 21 links, 20 joints
Joints:
- removed joint base_link-base_fixed_joint
- removed joint base_link-base_link_inertia
- removed joint flange-tool0
- removed joint wrist_3-flange
- added joint base_link_base_fixed_joint: type fixed, parent base_link, child base, origin xyz=0 0 0 rpy=0 0 3.141592653589793
- added joint base_link_base_link_inertia: type fixed, parent base_link, child base_link_inertia, origin xyz=0 0 0 rpy=0 0 3.141592653589793
- added joint flange_tool0: type fixed, parent flange, child tool0, origin xyz=0 0 0 rpy=1.5707963267948966 0 1.5707963267948966
- added joint wrist_3_flange: type fixed, parent wrist_3_link, child flange, origin xyz=0 0 0 rpy=0 -1.5707963267948966 -1.5707963267948966
